File: circuit/circuit.brd (EAGLE design)
At the start: 119.8 x 95.2 mm, 114 parts, among them IC2 MAX232ECWE, IC3 L298, IC4 L298, IC5 L298, IC6 74AC04D, IC7 ATMEGA64-SOCKEL, T1 BC 548B, T2 BC 548B, T3 BC 548B, X1 MICROMATCH-4, X2 MICROMATCH-8

Commit message: update to Version 7.0.2
Routing:
- net N$25: track 0.00 -> 5.08 mm
- net N$22: track 0.00 -> 5.08 mm
- net N$23: track 0.00 -> 2.54 mm
Other:
- board text added: "26.11.2014"
- board text added: "Boot"
- board text added: "RS232"
- board text added: "TX"
- board text added: "V 7.0.2"
- board text removed: "25.11.2014"
- board text removed: "V 7.0.1"
